File: template_v1.0/stm32_base.kicad_sch (KiCad schematic)
At the start: 49 parts, among them J1 Network Connector, J2 STDC14, SW1 SW_Push, U1 LD39050PU33R, U2 STM32G474RBT6, U3 TJA1042T-3, Y1 8MHz

Commit message: Add 24 V to 5 V Voltage Regulator
Parts:
- removed C1, C6: 100n, Capacitor_SMD:C_0402_1005Metric, symbol Device:C
- removed C4, C5: 1u, Capacitor_SMD:C_0402_1005Metric, symbol Device:C
- removed U1: LD39050PU33R, Package_DFN_QFN:DFN-6-1EP_3x3mm_P0.95mm_EP1.7x2.6mm, symbol Exocet:LD39050PU33R
- added U1: TSR1-2450E, Converter_DCDC:Converter_DCDC_TRACO_TSR1-xxxxE_THT, symbol Converter_DCDC:TSR1-2450E
Connections:
- net +24V: now also U1.1 (Vin)
- net GND: now also U1.2 (GND)
- net +5V renamed 5V VDC
- net 5V VDC: now also U1.3 (Vout)
- no-connect marks 41 -> 40
Other:
- moved on the sheet: C19, D3, D4, D5, F2, J1, TP6, TP7
