File: template/stm32_base.kicad_sch (KiCad schematic)
At the start: 41 parts, among them J1 Network Connector, J2 STDC14, SW1 SW_Push, U1 LD39050PU33R, U2 STM32G474RBT6, U3 SN65HVD230, Y1 8MHz

Commit message: Removed copy folder, add schematic page with hierarchical reference
Parts:
- removed C5: 1u, Capacitor_SMD:C_0402_1005Metric, symbol Device:C
- removed C6: 100n, Capacitor_SMD:C_0402_1005Metric, symbol Device:C
- removed F1: 2A, Exocet:Fuse_Holder_Littelfuse_01530008, symbol Device:Fuse
- removed U1: LD39050PU33R, Package_DFN_QFN:DFN-6-1EP_3x3mm_P0.95mm_EP1.7x2.6mm, symbol Exocet:LD39050PU33R
- removed U3: SN65HVD230, Package_SO:SOIC-8_3.9x4.9mm_P1.27mm, symbol Interface_CAN_LIN:SN65HVD230
- added C18: 2.2uf, Capacitor_SMD:C_01005_0402Metric, symbol Device:C
- added C19: 10uf, Capacitor_SMD:C_0805_2012Metric, symbol Device:C
- added D3: SMF28A, Diode_SMD:D_SOD-123F, symbol Device:D_Zener
- added D4, D5: SMF4L24CA, Diode_SMD:D_SOD-123F, symbol Diode:1N630xCA
- added F2: 7.5, Exocet:Fuse_Holder_Littelfuse_01530008, symbol Device:Fuse
- added FB3: FerriteBead, Resistor_SMD:R_0805_2012Metric, symbol Device:FerriteBead
- added TP6: RED, Package_TO_SOT_SMD:SOT-23-5, symbol Connector:TestPoint
- added TP7: BLACK, symbol Connector:TestPoint
- added U1: TSR1-2450E, Converter_DCDC:Converter_DCDC_TRACO_TSR1-xxxxE_THT, symbol Converter_DCDC:TSR1-2450E
- added U3: TJA1042T-3, Package_SO:SOIC-8_3.9x4.9mm_P1.27mm, symbol Interface_CAN_LIN:TJA1042T-3
- added U4: LM3940, Package_TO_SOT_THT:TO-220-3_Vertical, symbol Exocet:LM3940
- C1: value 100n -> 0.47u; footprint Capacitor_SMD:C_0402_1005Metric -> Capacitor_SMD:C_0201_0603Metric; JLCPCB C1525 -> C1623
- C4: value 1u -> 47uf; footprint Capacitor_SMD:C_0402_1005Metric -> Capacitor_Tantalum_SMD:CP_EIA-3216-10_Kemet-I; JLCPCB C52923 -> C7190
- C9: footprint Capacitor_SMD:C_0402_1005Metric -> Package_SO:SOIC-8_3.9x4.9mm_P1.27mm; JLCPCB C1525 -> (none)
- R3: value 10k -> 1k; footprint Resistor_SMD:R_0402_1005Metric -> (none); JLCPCB C25744 -> (none)
Connections:
- net +24V: now also C19.1, D3.1 (K), F2.2, TP6.1, U1.1 (Vin); no longer J1.1 (+24V)
- net +3.3V: now also C4.1, FB3.1, U3.5 (VIO), U4.3 (OUT); no longer C7.1, C8.1, C9.1, U2.29 (VDDA)
- net CAN_H: now also J1.3 (CAN_H), D5.2 (A2), U3.7 (CANH); no longer J1.4 (CAN_H)
- net CAN_L: now also J1.2 (CAN_L), D4.2 (A2), U3.6 (CANL); no longer J1.3 (CAN_L)
- net CAN_RX: now also U3.4 (RXD)
- net CAN_TX: now also U3.1 (TXD)
- net GND: now also C9.1, J1.4 (GND), C18.2, C19.2, D3.2 (A), D4.1 (A1), D5.1 (A1), TP7.1, U1.2 (GND), U3.2 (GND), U4.2 (GND); no longer C9.2, J1.5 (GND), U2.27 (VSSA)
- net T_NRST: now also C18.1; no longer SW1.1
- net at R3.1: now also U3.8 (STB)
- net +5V renamed 5V VDC
- net 5V VDC: now also C9.2, U1.3 (Vout), U3.3 (VCC), U4.1 (IN); no longer C4.1
- new net: C7.1, C8.1, FB3.2, U2.29 (VDDA)
- new net: F2.1, J1.1 (+24V)
- no-connect marks 42 -> 40
Other:
- company: (none) -> Exocet Polytechnique Montréal
- moved on the sheet: C2, C3, C7, C8

Commit message: Implement review comments
Parts:
- removed TP5: TestPoint, TestPoint:TestPoint_Keystone_5005-5009_Compact, symbol Connector:TestPoint
- added C5: 100n, Capacitor_SMD:C_0402_1005Metric, symbol Device:C
- added D6: D, symbol Device:D
- added R6: 100, symbol Device:R
- C1: value 0.47u -> 470n
- C18: renamed from C17; value 100n -> 2.2u
- C4: value 47uf -> 47u; footprint Capacitor_Tantalum_SMD:CP_EIA-3216-10_Kemet-I -> (none); JLCPCB C7190 -> (none)
- F2: value 7.5 -> 5
- H1, H2, H3, H4: value 2.7mm -> M3; footprint MountingHole:MountingHole_2.7mm_Pad -> MountingHole:MountingHole_3.2mm_M3
- R4, R5: value 100 -> 1k
- U4: now not fitted
Connections:
- net 5V VDC: no longer C1.1, U1.3 (Vout), U4.1 (IN)
- net GND: now also C18.2, U2.27 (VSSA), C5.2, R6.2; no longer C18.1, C4.2, SW1.2
- net T_NRST: now also D6.2 (A); no longer C18.2
- net at SW1.1: now also C18.1, D6.1 (K)
- new net: R6.1, SW1.2
- new net: C4.2, C5.1
- new net +5V: C1.1, U1.3 (Vout), U4.1 (IN)
Other:
- note added: "Voltage Regulator 1"
- note added: "Voltage Regulator 2"
- note removed: "Voltage Regulator"
- moved on the sheet: C1, C18, C4, SW1, TP1, TP3, U1

Commit message: schem: move a few passives and change some fields
Parts:
- removed D6: D, symbol Device:D
- removed TP3: TestPoint, TestPoint:TestPoint_Keystone_5005-5009_Compact, symbol Connector:TestPoint
- added D3: SMF6.0A, Diode_SMD:D_SOD-123F, symbol Device:D_Zener
- added F1: Polyfuse, symbol Device:Polyfuse
- added Q1: Q_NMOS_DGS, symbol Transistor_FET:Q_NMOS_DGS
- added R5: 1.2k, Resistor_SMD:R_0402_1005Metric, symbol Device:R
- added R6: 100, Resistor_SMD:R_0402_1005Metric, symbol Device:R
- added TP5: RED, Package_TO_SOT_SMD:SOT-23-5, symbol Connector:TestPoint
- C17: renamed from C19; value 10uf -> 10u
- C18: value 2.2uf -> 100n; footprint Capacitor_SMD:C_01005_0402Metric -> Capacitor_SMD:C_0402_1005Metric; JLCPCB C12530 -> (none)
- C3: renamed from C1; footprint Capacitor_SMD:C_0201_0603Metric -> Capacitor_SMD:C_0603_1608Metric
- C4: symbol Device:C -> Device:C_Polarized
- D4, D5: value SMF4L24CA -> SMF4L48CA; JLCPCB C53278608 -> (none)
- D6: renamed from D3; value SMF28A -> SMF33A; JLCPCB C41376091 -> (none)
- H4: footprint MountingHole:MountingHole_3.2mm_M3 -> MountingHole:MountingHole_3.2mm_M3_Pad
- J1: footprint Connector_Molex:Molex_SPOX_5268-05A_1x05_P2.50mm_Horizontal -> (none); JLCPCB C185201 -> (none)
- SW1: now fitted
- TP1: renamed from TP2; MFR (none) -> Keystone; now fitted
- TP2: renamed from TP1; MFR (none) -> Keystone; now fitted
- TP3: renamed from TP4; MFR (none) -> Keystone; now fitted
- TP4: renamed from TP6; MFR (none) -> Keystone
- TP6: renamed from TP7; MFR (none) -> Keystone
- U1: MFR (none) -> Traco Power; MPN (none) -> TSR1-2450E
- U3: renamed from U4; JLCPCB C544820 -> (none); MFR (none) -> Texas Instruments; MPN (none) -> LM3940IT-3.3; now fitted
- renumbered C2 to C1, C11 to C10, C12 to C11, C13 to C12, C14 to C13, C15 to C14, C16 to C15, C18 to C16, C3 to C2, C7 to C6, C8 to C7, C9 to C8, C10 to C9, FB3 to FB1, R5 to R7, R6 to R8, U3 to U4
Connections:
- net +24V: now also C18.1
- net +3.3V: now also C5.1
- net +5V: now also R7.1, F1.2, TP5.1; no longer U1.3 (Vout)
- net GND: now also C4.2, D3.2 (A), Q1.3 (S), R5.2; no longer D2.1 (K)
- net STATUS_LED: now also R5.1, R6.1; no longer R7.1
- net T_NRST: now also C16.1, SW1.1, D3.1 (K); no longer C18.1
- new net: D2.1 (K), Q1.1 (D)
- new net: Q1.2 (G), R6.2
- new net: F1.1, U1.3 (Vout)
Other:
- moved on the sheet: C5, D2, FB1, R7, TP4
